File: preample/preample.sch (KiCad schematic (older format))
At the start: 67 parts, among them J1 Conn_01x03, J2 Conn_01x07, J3 Conn_01x06, SW1 SW_DPDT_x2, U1 TPS7A39, U2 OPA2134UA, U3 OPA134UA, U4 OPA2134UA, U5 OPA134UA

Commit message: Fixed cap issue in schematic. finished pcb layout
Parts:
- J1: footprint (none) -> Connector_JST:JST_PH_B3B-PH-K_1x03_P2.00mm_Vertical; Part No (none) -> B3B-PH-K-S(LF)(SN)
- J2: footprint (none) -> Connector_JST:JST_PH_B7B-PH-K_1x07_P2.00mm_Vertical; Part No (none) -> B7B-PH-K-S(LF)(SN)
- J3: footprint (none) -> Connector_JST:JST_PH_B6B-PH-K_1x06_P2.00mm_Vertical; Part No (none) -> B6B-PH-K-S(LF)(SN)
Connections:
- net +24V: now also C1.1; no longer C1.2
- net -24V: now also C2.2, C4.2; no longer C2.1, C4.1
- net GND: now also C1.2, C2.1, C4.1; no longer C1.1, C2.2, C4.2
- net TRIM_1A: now also RV2.3; no longer RV2.1
- net TRIM_1B: now also RV2.1; no longer RV2.3
- net TRIM_2A: now also RV3.3; no longer RV3.1
- net TRIM_2B: now also RV3.1; no longer RV3.3
- net at J1.1 (Pin_1): now also R1.2; no longer R2.1
- net at J1.3 (Pin_3): now also R2.1; no longer R1.2
Other:
- moved on the sheet: C1, C2, R1, R2
Changed lines of the file:
@@
 F 4 "CL31B106KBHNNNE" H 2800 2600 50  0001 C CNN "Part No"
 	1    2800 2600
-	1    0    0    -1
+	-1   0    0    1
 $EndComp
 $Comp
@@
 	1    0    0    -1
 $EndComp
-Wire Wire Line
-	2800 2500 2650 2500
-Connection ~ 2800 2500
 $Comp
 L Device:CP1_Small C9
@@
 F 0 "J1" V 1450 1000 50  0000 C CNN
 F 1 "Conn_01x03" V 1550 1000 50  0000 C CNN
-F 2 "" H 1350 1000 50  0001 C CNN
+F 2 "Connector_JST:JST_PH_B3B-PH-K_1x03_P2.00mm_Vertical" H 1350 1000 50  0001 C CNN
 F 3 "~" H 1350 1000 50  0001 C CNN
+F 4 "B3B-PH-K-S(LF)(SN)" V 1350 1000 50  0001 C CNN "Part No"
 	1    1350 1000
 	0    -1   -1   0
@@
 L power:+24V #PWR0103
 U 1 1 5CC43794
-P 650 1100
-F 0 "#PWR0103" H 650 950 50  0001 C CNN
-F 1 "+24V" H 665 1273 50  0000 C CNN
-F 2 "" H 650 1100 50  0001 C CNN
-F 3 "" H 650 1100 50  0001 C CNN
-	1    650  1100
+P 1950 1100
+F 0 "#PWR0103" H 1950 950 50  0001 C CNN
+F 1 "+24V" H 1965 1273 50  0000 C CNN
+F 2 "" H 1950 1100 50  0001 C CNN
+F 3 "" H 1950 1100 50  0001 C CNN
+	1    1950 1100
 	1    0    0    -1
 $EndComp
@@
 L power:-24V #PWR0104
 U 1 1 5CC45A35
-P 2000 1100
-F 0 "#PWR0104" H 2000 1200 50  0001 C CNN
-F 1 "-24V" H 2015 1273 50  0000 C CNN
-F 2 "" H 2000 1100 50  0001 C CNN
-F 3 "" H 2000 1100 50  0001 C CNN
-	1    2000 1100
+P 750 1100
+F 0 "#PWR0104" H 750 1200 50  0001 C CNN
+F 1 "-24V" H 765 1273 50  0000 C CNN
+F 2 "" H 750 1100 50  0001 C CNN
+F 3 "" H 750 1100 50  0001 C CNN
+	1    750  1100
 	1    0    0    -1
 $EndComp
@@
 L Device:R_Small_US R2
 U 1 1 5CC61DFA
-P 950 1300
-F 0 "R2" V 745 1300 50  0000 C CNN
-F 1 "3R" V 836 1300 50  0000 C CNN
-F 2 "Resistor_SMD:R_0805_2012Metric" H 950 1300 50  0001 C CNN
-F 3 "~" H 950 1300 50  0001 C CNN
-F 4 "ERJ-6DQF3R3V" V 950 1300 50  0001 C CNN "Part No"
-	1    950  1300
-	0    1    1    0
-$EndComp
-$Comp
-L Device:CP1_Small C2
-U 1 1 5CC679C1
-P 2000 1450
-F 0 "C2" H 2091 1496 50  0000 L CNN
-F 1 "680uF" H 2091 1405 50  0000 L CNN
-F 2 "preample:EEV-FK1H681M" H 2000 1450 50  0001 C CNN
-F 3 "~" H 2000 1450 50  0001 C CNN
-F 4 "EEV-FK1H681M" H 2000 1450 50  0001 C CNN "Part No"
-	1    2000 1450
-	1    0    0    -1
-$EndComp
-$Comp
-L Device:CP1_Small C1
-U 1 1 5CC69634
-P 650 1450
-F 0 "C1" H 450 1400 50  0000 L CNN
-F 1 "680uF" H 300 1500 50  0000 L CNN
-F 2 "preample:EEV-FK1H681M" H 650 1450 50  0001 C CNN
-F 3 "~" H 650 1450 50  0001 C CNN
-F 4 "EEV-FK1H681M" H 650 1450 50  0001 C CNN "Part No"
-	1    650  1450
-	-1   0    0    1
-$EndComp
-Wire Wire Line
-	2000 1100 2000 1300
-Wire Wire Line
-	2000 1300 1800 1300
-Connection ~ 2000 1300
-Wire Wire Line
-	2000 1300 2000 1350
-Wire Wire Line
-	1600 1300 1450 1300
-Wire Wire Line
-	1450 1300 1450 1200
-Wire Wire Line
-	1350 1200 1350 1600
-Wire Wire Line
-	2000 1550 2000 1600
-Wire Wire Line
-	1250 1200 1250 1300
-Wire Wire Line
-	1250 1300 1050 1300
-Wire Wire Line
-	850  1300 650  1300
-Wire Wire Line
-	650  1300 650  1100
-Wire Wire Line
-	650  1300 650  1350
-Connection ~ 650  1300
-Wire Wire Line
-	650  1550 650  1600
-$Comp
-L Device:R_Small_US R1
-U 1 1 5CC611FD
 P 1700 1300
-F 0 "R1" V 1495 1300 50  0000 C CNN
-F 1 "3R" V 1586 1300 50  0000 C CNN
+F 0 "R2" V 1900 1300 50  0000 C CNN
+F 1 "3R" V 1800 1300 50  0000 C CNN
 F 2 "Resistor_SMD:R_0805_2012Metric" H 1700 1300 50  0001 C CNN
 F 3 "~" H 1700 1300 50  0001 C CNN
 F 4 "ERJ-6DQF3R3V" V 1700 1300 50  0001 C CNN "Part No"
 	1    1700 1300
-	0    1    1    0
+	0    -1   -1   0
+$EndComp
+$Comp
+L Device:CP1_Small C2
+U 1 1 5CC679C1
+P 750 1450
+F 0 "C2" H 500 1450 50  0000 L CNN
+F 1 "680uF" H 400 1550 50  0000 L CNN
+F 2 "preample:EEV-FK1H681M" H 750 1450 50  0001 C CNN
+F 3 "~" H 750 1450 50  0001 C CNN
+F 4 "EEV-FK1H681M" H 750 1450 50  0001 C CNN "Part No"
+	1    750  1450
+	-1   0    0    1
+$EndComp
+$Comp
+L Device:CP1_Small C1
+U 1 1 5CC69634
+P 1950 1450
+F 0 "C1" H 1700 1450 50  0000 L CNN
+F 1 "680uF" H 1600 1350 50  0000 L CNN
+F 2 "preample:EEV-FK1H681M" H 1950 1450 50  0001 C CNN
+F 3 "~" H 1950 1450 50  0001 C CNN
+F 4 "EEV-FK1H681M" H 1950 1450 50  0001 C CNN "Part No"
+	1    1950 1450
+	1    0    0    -1
+$EndComp
+Wire Wire Line
+	750  1100 750  1300
+Connection ~ 750  1300
+Wire Wire Line
+	750  1300 750  1350
+Wire Wire Line
+	1450 1300 1450 1200
+Wire Wire Line
+	1350 1200 1350 1600
+Wire Wire Line
+	750  1550 750  1600
+Wire Wire Line
+	1250 1200 1250 1300
+Wire Wire Line
+	1950 1550 1950 1600
+$Comp
+L Device:R_Small_US R1
+U 1 1 5CC611FD
+P 1000 1300
+F 0 "R1" V 1200 1300 50  0000 C CNN
+F 1 "3R" V 1100 1300 50  0000 C CNN
+F 2 "Resistor_SMD:R_0805_2012Metric" H 1000 1300 50  0001 C CNN
+F 3 "~" H 1000 1300 50  0001 C CNN
+F 4 "ERJ-6DQF3R3V" V 1000 1300 50  0001 C CNN "Part No"
+	1    1000 1300
+	0    -1   -1   0
 $EndComp
 Wire Wire Line
@@
 	4350 1300 4300 1300
 Wire Wire Line
-	2800 2500 3050 2500
-Wire Wire Line
 	3050 2500 3050 3100
 Connection ~ 3050 2500
@@
 Wire Wire Line
 	8750 4100 8850 4100
+Text GLabel 10750 4400 3    50   Input ~ 0
+TRIM_2A
 Text GLabel 10250 4400 3    50   Input ~ 0
-TRIM_2A
-Text GLabel 10750 4400 3    50   Input ~ 0
 TRIM_2B
+Text GLabel 9500 4400 3    50   Input ~ 0
+TRIM_1A
 Text GLabel 9000 4400 3    50   Input ~ 0
-TRIM_1A
-Text GLabel 9500 4400 3    50   Input ~ 0
 TRIM_1B
 Wire Wire Line
@@
 F 0 "J2" H 7980 4442 50  0000 L CNN
 F 1 "Conn_01x07" H 7980 4351 50  0000 L CNN
-F 2 "" H 7900 4400 50  0001 C CNN
+F 2 "Connector_JST:JST_PH_B7B-PH-K_1x07_P2.00mm_Vertical" H 7900 4400 50  0001 C CNN
 F 3 "~" H 7900 4400 50  0001 C CNN
+F 4 "B7B-PH-K-S(LF)(SN)" H 7900 4400 50  0001 C CNN "Part No"
 	1    7900 4400
 	1    0    0    -1
@@
 L power:GNDREF #AUXGND0102
 U 1 1 5CDF235A
-P 650 1600
-F 0 "#AUXGND0102" H 738 1563 50  0001 L CNN
-F 1 "GNDREF" H 655 1427 50  0000 C CNN
-F 2 "" H 650 1600 50  0001 C CNN
-F 3 "" H 650 1600 50  0001 C CNN
-	1    650  1600
+P 1950 1600
+F 0 "#AUXGND0102" H 2038 1563 50  0001 L CNN
+F 1 "GNDREF" H 1955 1427 50  0000 C CNN
+F 2 "" H 1950 1600 50  0001 C CNN
+F 3 "" H 1950 1600 50  0001 C CNN
+	1    1950 1600
 	1    0    0    -1
 $EndComp
@@
 L power:GNDREF #AUXGND0103
 U 1 1 5CDFFCF5
-P 2000 1600
-F 0 "#AUXGND0103" H 2088 1563 50  0001 L CNN
-F 1 "GNDREF" H 2005 1427 50  0000 C CNN
-F 2 "" H 2000 1600 50  0001 C CNN
-F 3 "" H 2000 1600 50  0001 C CNN
-	1    2000 1600
+P 750 1600
+F 0 "#AUXGND0103" H 838 1563 50  0001 L CNN
+F 1 "GNDREF" H 755 1427 50  0000 C CNN
+F 2 "" H 750 1600 50  0001 C CNN
+F 3 "" H 750 1600 50  0001 C CNN
+	1    750  1600
 	1    0    0    -1
 $EndComp
@@
 U 1 1 5CD108C4
 P 9200 950
-F 0 "SW1" H 9200 625 50  0000 C CNN
-F 1 "SW_DPDT_x2" H 9200 716 50  0000 C CNN
+F 0 "SW1" H 9200 1250 50  0000 C CNN
+F 1 "SW_DPDT_x2" H 9200 1150 50  0000 C CNN
 F 2 "preample:PBH2UEENAGX" H 9200 950 50  0001 C CNN
 F 3 "~" H 9200 950 50  0001 C CNN
@@
 F 0 "J3" H 6968 775 50  0000 C CNN
 F 1 "Conn_01x06" H 6968 866 50  0000 C CNN
-F 2 "" H 7050 1300 50  0001 C CNN
+F 2 "Connector_JST:JST_PH_B6B-PH-K_1x06_P2.00mm_Vertical" H 7050 1300 50  0001 C CNN
 F 3 "~" H 7050 1300 50  0001 C CNN
+F 4 "B6B-PH-K-S(LF)(SN)" H 7050 1300 50  0001 C CNN "Part No"
 	1    7050 1300
 	-1   0    0    1
@@
 	0    -1   -1   0
 $EndComp
+Wire Wire Line
+	1950 1100 1950 1300
+Connection ~ 1950 1300
+Wire Wire Line
+	1950 1300 1950 1350
+Wire Wire Line
+	1450 1300 1600 1300
+Wire Wire Line
+	1800 1300 1950 1300
+Wire Wire Line
+	1100 1300 1250 1300
+Wire Wire Line
+	900  1300 750  1300
+Wire Wire Line
+	2650 2500 2800 2500
+Connection ~ 2800 2500
+Wire Wire Line
+	2800 2500 3050 2500
 $EndSCHEMATC

Commit message: Changes resistors for opamps to 0805s. Chose more realistic power resistors. rerouted for new components.
Parts:
- R1, R2: value 3R -> 15R; footprint Resistor_SMD:R_0805_2012Metric -> Resistor_SMD:R_2512_6332Metric; Part No ERJ-6DQF3R3V -> RPC2512JT15R0
- R10, R11, R12, R16, R17, R18, R19, R9: value 560R -> 5K6; footprint Resistor_SMD:R_0402_1005Metric -> Resistor_SMD:R_0805_2012Metric
- R13, R14, R15, R20, R21, R22, R23, R7, R8: footprint Resistor_SMD:R_0402_1005Metric -> Resistor_SMD:R_0805_2012Metric
Changed lines of the file:
@@
 P 1700 1300
 F 0 "R2" V 1900 1300 50  0000 C CNN
-F 1 "3R" V 1800 1300 50  0000 C CNN
-F 2 "Resistor_SMD:R_0805_2012Metric" H 1700 1300 50  0001 C CNN
+F 1 "15R" V 1800 1300 50  0000 C CNN
+F 2 "Resistor_SMD:R_2512_6332Metric" H 1700 1300 50  0001 C CNN
 F 3 "~" H 1700 1300 50  0001 C CNN
-F 4 "ERJ-6DQF3R3V" V 1700 1300 50  0001 C CNN "Part No"
+F 4 "RPC2512JT15R0" V 1700 1300 50  0001 C CNN "Part No"
 	1    1700 1300
 	0    -1   -1   0
@@
 P 1000 1300
 F 0 "R1" V 1200 1300 50  0000 C CNN
-F 1 "3R" V 1100 1300 50  0000 C CNN
-F 2 "Resistor_SMD:R_0805_2012Metric" H 1000 1300 50  0001 C CNN
+F 1 "15R" V 1100 1300 50  0000 C CNN
+F 2 "Resistor_SMD:R_2512_6332Metric" H 1000 1300 50  0001 C CNN
 F 3 "~" H 1000 1300 50  0001 C CNN
-F 4 "ERJ-6DQF3R3V" V 1000 1300 50  0001 C CNN "Part No"
+F 4 "RPC2512JT15R0" V 1000 1300 50  0001 C CNN "Part No"
 	1    1000 1300
 	0    -1   -1   0
@@
 	5200 6900 5200 7000
 $Comp
-L Device:R_Small_US R11
-U 1 1 5CCD5D27
-P 5300 3650
-F 0 "R11" V 5095 3650 50  0000 C CNN
-F 1 "560R" V 5186 3650 50  0000 C CNN
-F 2 "Resistor_SMD:R_0402_1005Metric" H 5300 3650 50  0001 C CNN
-F 3 "~" H 5300 3650 50  0001 C CNN
-	1    5300 3650
-	0    1    1    0
-$EndComp
-$Comp
 L Device:R_Small_US R13
 U 1 1 5CCD7640
@@
 F 0 "R13" V 6205 4350 50  0000 C CNN
 F 1 "47R" V 6114 4350 50  0000 C CNN
-F 2 "Resistor_SMD:R_0402_1005Metric" H 6000 4350 50  0001 C CNN
+F 2 "Resistor_SMD:R_0805_2012Metric" H 6000 4350 50  0001 C CNN
 F 3 "~" H 6000 4350 50  0001 C CNN
 	1    6000 4350
@@
 P 4800 4250
 F 0 "R9" V 4595 4250 50  0000 C CNN
-F 1 "560R" V 4686 4250 50  0000 C CNN
-F 2 "Resistor_SMD:R_0402_1005Metric" H 4800 4250 50  0001 C CNN
+F 1 "5K6" V 4686 4250 50  0000 C CNN
+F 2 "Resistor_SMD:R_0805_2012Metric" H 4800 4250 50  0001 C CNN
 F 3 "~" H 4800 4250 50  0001 C CNN
 	1    4800 4250
@@
 P 4800 4450
 F 0 "R10" V 4700 4400 50  0000 L CNN
-F 1 "560R" V 4600 4400 50  0000 L CNN
-F 2 "Resistor_SMD:R_0402_1005Metric" H 4800 4450 50  0001 C CNN
+F 1 "5K6" V 4600 4400 50  0000 L CNN
+F 2 "Resistor_SMD:R_0805_2012Metric" H 4800 4450 50  0001 C CNN
 F 3 "~" H 4800 4450 50  0001 C CNN
 	1    4800 4450
@@
 P 5250 5900
 F 0 "R18" V 5045 5900 50  0000 C CNN
-F 1 "560R" V 5136 5900 50  0000 C CNN
-F 2 "Resistor_SMD:R_0402_1005Metric" H 5250 5900 50  0001 C CNN
+F 1 "5K6" V 5136 5900 50  0000 C CNN
+F 2 "Resistor_SMD:R_0805_2012Metric" H 5250 5900 50  0001 C CNN
 F 3 "~" H 5250 5900 50  0001 C CNN
 	1    5250 5900
@@
 P 4750 6500
 F 0 "R16" V 4545 6500 50  0000 C CNN
-F 1 "560R" V 4636 6500 50  0000 C CNN
-F 2 "Resistor_SMD:R_0402_1005Metric" H 4750 6500 50  0001 C CNN
+F 1 "5K6" V 4636 6500 50  0000 C CNN
+F 2 "Resistor_SMD:R_0805_2012Metric" H 4750 6500 50  0001 C CNN
 F 3 "~" H 4750 6500 50  0001 C CNN
 	1    4750 6500
@@
 P 4750 6700
 F 0 "R17" V 4650 6700 50  0000 C CNN
-F 1 "560R" V 4550 6700 50  0000 C CNN
-F 2 "Resistor_SMD:R_0402_1005Metric" H 4750 6700 50  0001 C CNN
+F 1 "5K6" V 4550 6700 50  0000 C CNN
+F 2 "Resistor_SMD:R_0805_2012Metric" H 4750 6700 50  0001 C CNN
 F 3 "~" H 4750 6700 50  0001 C CNN
 	1    4750 6700
@@
 P 4950 7200
 F 0 "R19" H 4882 7154 50  0000 R CNN
-F 1 "560R" H 4882 7245 50  0000 R CNN
-F 2 "Resistor_SMD:R_0402_1005Metric" H 4950 7200 50  0001 C CNN
+F 1 "5K6" H 4882 7245 50  0000 R CNN
+F 2 "Resistor_SMD:R_0805_2012Metric" H 4950 7200 50  0001 C CNN
 F 3 "~" H 4950 7200 50  0001 C CNN
 	1    4950 7200
@@
 F 0 "R21" H 7968 5796 50  0000 L CNN
 F 1 "100R" H 7968 5705 50  0000 L CNN
-F 2 "Resistor_SMD:R_0402_1005Metric" H 7900 5750 50  0001 C CNN
+F 2 "Resistor_SMD:R_0805_2012Metric" H 7900 5750 50  0001 C CNN
 F 3 "~" H 7900 5750 50  0001 C CNN
 	1    7900 5750
@@
 F 0 "R7" H 1382 4254 50  0000 R CNN
 F 1 "47K" H 1382 4345 50  0000 R CNN
-F 2 "Resistor_SMD:R_0402_1005Metric" H 1450 4300 50  0001 C CNN
+F 2 "Resistor_SMD:R_0805_2012Metric" H 1450 4300 50  0001 C CNN
 F 3 "~" H 1450 4300 50  0001 C CNN
 	1    1450 4300
@@
 F 0 "R14" H 1382 6504 50  0000 R CNN
 F 1 "47K" H 1382 6595 50  0000 R CNN
-F 2 "Resistor_SMD:R_0402_1005Metric" H 1450 6550 50  0001 C CNN
+F 2 "Resistor_SMD:R_0805_2012Metric" H 1450 6550 50  0001 C CNN
 F 3 "~" H 1450 6550 50  0001 C CNN
 	1    1450 6550
@@
 F 0 "R20" V 5795 6600 50  0000 C CNN
 F 1 "47R" V 5886 6600 50  0000 C CNN
-F 2 "Resistor_SMD:R_0402_1005Metric" H 6000 6600 50  0001 C CNN
+F 2 "Resistor_SMD:R_0805_2012Metric" H 6000 6600 50  0001 C CNN
 F 3 "~" H 6000 6600 50  0001 C CNN
 	1    6000 6600
@@
 F 0 "R22" V 1000 4100 50  0000 R CNN
 F 1 "1K" V 900 4050 50  0000 R CNN
-F 2 "Resistor_SMD:R_0402_1005Metric" H 1100 4000 50  0001 C CNN
+F 2 "Resistor_SMD:R_0805_2012Metric" H 1100 4000 50  0001 C CNN
 F 3 "~" H 1100 4000 50  0001 C CNN
 	1    1100 4000
@@
 F 0 "R23" V 1000 6350 50  0000 R CNN
 F 1 "1K" V 900 6300 50  0000 R CNN
-F 2 "Resistor_SMD:R_0402_1005Metric" H 1100 6250 50  0001 C CNN
+F 2 "Resistor_SMD:R_0805_2012Metric" H 1100 6250 50  0001 C CNN
 F 3 "~" H 1100 6250 50  0001 C CNN
 	1    1100 6250
@@
 P 5000 4950
 F 0 "R12" H 4932 4904 50  0000 R CNN
-F 1 "560R" H 4932 4995 50  0000 R CNN
-F 2 "Resistor_SMD:R_0402_1005Metric" H 5000 4950 50  0001 C CNN
+F 1 "5K6" H 4932 4995 50  0000 R CNN
+F 2 "Resistor_SMD:R_0805_2012Metric" H 5000 4950 50  0001 C CNN
 F 3 "~" H 5000 4950 50  0001 C CNN
 	1    5000 4950
@@
 F 0 "R8" V 2000 4600 50  0000 R CNN
 F 1 "1K" V 1900 4550 50  0000 R CNN
-F 2 "Resistor_SMD:R_0402_1005Metric" H 2100 4500 50  0001 C CNN
+F 2 "Resistor_SMD:R_0805_2012Metric" H 2100 4500 50  0001 C CNN
 F 3 "~" H 2100 4500 50  0001 C CNN
 	1    2100 4500
@@
 F 0 "R15" V 2000 6850 50  0000 R CNN
 F 1 "1K" V 1900 6800 50  0000 R CNN
-F 2 "Resistor_SMD:R_0402_1005Metric" H 2100 6750 50  0001 C CNN
+F 2 "Resistor_SMD:R_0805_2012Metric" H 2100 6750 50  0001 C CNN
 F 3 "~" H 2100 6750 50  0001 C CNN
 	1    2100 6750
@@
 Wire Wire Line
 	2800 2500 3050 2500
+$Comp
+L Device:R_Small_US R11
+U 1 1 5CCD5D27
+P 5300 3650
+F 0 "R11" V 5095 3650 50  0000 C CNN
+F 1 "5K6" V 5186 3650 50  0000 C CNN
+F 2 "Resistor_SMD:R_0805_2012Metric" H 5300 3650 50  0001 C CNN
+F 3 "~" H 5300 3650 50  0001 C CNN
+	1    5300 3650
+	0    1    1    0
+$EndComp
 $EndSCHEMATC

Commit message: Added simulation. Added current path for negative feed forward cap. Chose resistors for amplifier circuits.
Parts:
- added D4: D_Schottky_ALT, Diode_SMD:D_SOD-323F, symbol Device:D_Schottky_ALT
- R10, R11, R12, R16, R17, R18, R19, R9: value 5K6 -> 11K5; Part No (none) -> ERA-6AEB1152V
- R13, R20: Part No (none) -> ERA-6AEB470V
- R14, R7: Part No (none) -> ERA-6AEB473V
- R15, R22, R23, R8: Part No (none) -> ERA-6AEB102V
- R21: Part No (none) -> ERA-6AEB101V
Connections:
- net GND: now also D4.1 (K)
- net at C9.1, R5.1, R6.2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: now also D4.2 (A)
- no-connect marks 0 -> 3
Other:
- note added: "CHANNEL 1 = LEFT CHANNEL\nCHANNEL 2 = RIGHT CHANNEL"
