File: power/power.kicad_pcb (KiCad board)
At the start: 2 copper layers, 36 x 34 mm, 5 parts, among them J1 Conn_01x02_Female, J2 Conn_01x02_Female, SW1 SW_DPST

Commit message: Reorganized repo. Added gerbers.
Parts:
- added F1: Fuse_Small, power:Keystone 4628 Fuse Holder, F.Cu at (88.8, 52.0)
Connections:
- J1 pad 1: Net-(J1-Pad1) -> Net-(F1-Pad2)
- SW1 pad 1: Net-(J1-Pad1) -> Net-(F1-Pad1)
Routing:
- net Net-(J1-Pad1): track 22.2 -> 0.00 mm
- net Net-(F1-Pad2): track 0.00 -> 21.3 mm
- net Net-(F1-Pad1): track 0.00 -> 20.9 mm
Other:
- outline, holes or cut-outs redrawn
- board text added: "HOT"
