File: power/power.sch (KiCad schematic (older format))
At the start: 3 parts, among them J1 Conn_01x02_Female, J2 Conn_01x02_Female, SW1 SW_DPST

Commit message: Reorganized repo. Added gerbers.
Parts:
- added F1: Fuse_Small, power:Keystone 4628 Fuse Holder, symbol Device:Fuse_Small
Connections:
- net at SW1.1: now also F1.1; no longer J1.1 (Pin_1)
- new net: F1.2, J1.1 (Pin_1)
Changed lines of the file:
@@
 	4800 2950 4650 2950
-Wire Wire Line
-	4650 2950 4650 3200
 Wire Wire Line
 	5200 2950 5550 2950
@@
 	4800 2750 4550 2750
 Wire Wire Line
-	4550 2750 4550 3200
-Wire Wire Line
 	5450 2750 5450 3200
 Wire Wire Line
 	5550 2950 5550 3200
+$Comp
+L Device:Fuse_Small F1
+U 1 1 5CF31E3C
+P 4650 3050
+F 0 "F1" V 4604 3098 50  0000 L CNN
+F 1 "Fuse_Small" V 4695 3098 50  0000 L CNN
+F 2 "power:Keystone 4628 Fuse Holder" H 4650 3050 50  0001 C CNN
+F 3 "~" H 4650 3050 50  0001 C CNN
+	1    4650 3050
+	0    1    1    0
+$EndComp
+Wire Wire Line
+	4650 3200 4650 3150
+Wire Wire Line
+	4550 3200 4550 2750
 $EndSCHEMATC
